File: Lectores_DVD/PCB/smd_11/smd_11.brd (EAGLE design)
At the start: 47 x 34 mm, 2 parts, among them J1 52793-1170

Commit message: Actualizacion
Other:
- board size 47 x 34 mm -> 47 x 28.9 mm
Changed lines of the file:
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@@
 <board>
 <plain>
-<wire x1="0" y1="0" x2="46.97" y2="0" width="0" layer="20"/>
-<wire x1="46.97" y1="0" x2="46.97" y2="33.96" width="0" layer="20"/>
+<wire x1="0" y1="5.08" x2="46.97" y2="5.08" width="0" layer="20"/>
+<wire x1="46.97" y1="5.08" x2="46.97" y2="33.96" width="0" layer="20"/>
 <wire x1="46.97" y1="33.96" x2="0" y2="33.96" width="0" layer="20"/>
-<wire x1="0" y1="33.96" x2="0" y2="0" width="0" layer="20"/>
-<hole x="3.81" y="3.81" drill="3"/>
+<wire x1="0" y1="33.96" x2="0" y2="5.08" width="0" layer="20"/>
+<hole x="3.81" y="8.89" drill="3"/>
 <hole x="3.81" y="29.21" drill="3"/>
 <hole x="41.91" y="29.21" drill="3"/>
-<hole x="41.91" y="3.81" drill="3"/>
+<hole x="41.91" y="8.89" drill="3"/>
 </plain>
 <attributes>
@@
 <signal name="GND">
 <polygon width="0.6096" layer="16">
-<vertex x="0" y="34.29"/>
-<vertex x="46.99" y="34.29"/>
-<vertex x="46.99" y="0"/>
-<vertex x="0" y="0"/>
+<vertex x="3.81" y="31.75"/>
+<vertex x="41.91" y="31.75"/>
+<vertex x="41.91" y="6.35"/>
+<vertex x="3.81" y="6.35"/>
 </polygon>
 <polygon width="0.6096" layer="1">
-<vertex x="0" y="34.29"/>
-<vertex x="0" y="0"/>
-<vertex x="46.99" y="0"/>
-<vertex x="46.99" y="34.29"/>
+<vertex x="3.81" y="31.75"/>
+<vertex x="3.81" y="6.35"/>
+<vertex x="41.91" y="6.35"/>
+<vertex x="41.91" y="31.75"/>
 </polygon>
-<via x="6.35" y="15.24" extent="1-16" drill="0.65"/>
+<via x="8.89" y="19.05" extent="1-16" drill="0.65"/>
 </signal>
 </signals>
