File: Lectores_DVD/PCB/smd_11_v2/smd_11.brd (EAGLE design)
At the start: 47 x 34 mm, 2 parts, among them J1 52793-1170

Commit message: Actualizacion
Parts:
- added U$1: (no value), logos_top:URJC
- added U$2: (no value), logos_top:LABTEL
Other:
- board size 47 x 34 mm -> 47 x 30.2 mm
Changed lines of the file:
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@@
 <board>
 <plain>
-<wire x1="0" y1="0" x2="46.97" y2="0" width="0" layer="20"/>
-<wire x1="46.97" y1="0" x2="46.97" y2="33.96" width="0" layer="20"/>
+<wire x1="0" y1="3.81" x2="46.97" y2="3.81" width="0" layer="20"/>
+<wire x1="46.97" y1="3.81" x2="46.97" y2="33.96" width="0" layer="20"/>
 <wire x1="46.97" y1="33.96" x2="0" y2="33.96" width="0" layer="20"/>
-<wire x1="0" y1="33.96" x2="0" y2="0" width="0" layer="20"/>
-<hole x="3.81" y="3.81" drill="3"/>
+<wire x1="0" y1="33.96" x2="0" y2="3.81" width="0" layer="20"/>
+<hole x="3.81" y="7.62" drill="3"/>
 <hole x="3.81" y="29.21" drill="3"/>
 <hole x="41.91" y="29.21" drill="3"/>
-<hole x="41.91" y="3.81" drill="3"/>
+<hole x="41.91" y="7.62" drill="3"/>
+<dimension x1="3.81" y1="29.21" x2="3.81" y2="34.29" x3="41.91" y3="31.75" textsize="1.778" layer="255"/>
 </plain>
 <attributes>
@@
 <attribute name="VALUE" x="8.89" y="27.178" size="0.6096" layer="27" font="vector" ratio="20"/>
 </element>
+<element name="U$1" library="logos_top" package="URJC" value="" x="6.35" y="15.24" smashed="yes"/>
+<element name="U$2" library="logos_top" package="LABTEL" value="" x="40.64" y="7.62" smashed="yes" rot="R90"/>
 </elements>
 <signals>
@@
 <signal name="GND">
 <polygon width="0.6096" layer="16">
-<vertex x="0" y="34.29"/>
-<vertex x="46.99" y="34.29"/>
-<vertex x="46.99" y="0"/>
-<vertex x="0" y="0"/>
+<vertex x="3.81" y="31.75"/>
+<vertex x="41.91" y="31.75"/>
+<vertex x="41.91" y="6.35"/>
+<vertex x="3.81" y="6.35"/>
 </polygon>
 <polygon width="0.6096" layer="1">
-<vertex x="0" y="34.29"/>
-<vertex x="0" y="0"/>
-<vertex x="46.99" y="0"/>
-<vertex x="46.99" y="34.29"/>
+<vertex x="3.81" y="31.75"/>
+<vertex x="3.81" y="6.35"/>
+<vertex x="41.91" y="6.35"/>
+<vertex x="41.91" y="31.75"/>
 </polygon>
 </signal>
@@
 <mfgpreviewcolor name="substratecolor" color="0xFF786E46"/>
 </mfgpreviewcolors>
+<errors>
+</errors>
 </board>
 </drawing>
